Commit message: Add localization stack: IMU link, EKF config, and separate sensor fusion launch file

File: src/warehouse_real_description/description/robot_core.xacro (robot description, xacro)
@@ -148,4 +148,18 @@
         <mu2 value="0.001"/>
     </gazebo>
+    <!-- IMU LINK -->
+    <link name="imu_link">
+    <visual>
+        <geometry>
+            <box size="0.01 0.01 0.01"/>
+        </geometry>
+        <material name="black"/>
+    </visual>
+    </link>
+    <joint name="imu_joint" type="fixed">
+        <parent link="base_link"/>
+        <child link="imu_link"/>
+        <origin xyz="0 0 0.05" rpy="0 0 0"/>
+    </joint>
     <!-- BACK CASTER WHEEL LINK -->
     <!-- <joint name="back_caster_wheel_joint" type="fixed">

Commit message: Add lifter joit and clean the diffdrive_arduino pkg

File: src/warehouse_real_description/description/robot_core.xacro (robot description, xacro)
@@ -162,4 +162,31 @@
         <origin xyz="0 0 0.05" rpy="0 0 0"/>
     </joint>
+    <link name="lifter_link">
+        <visual>
+            <origin xyz="0 0 0" rpy="0 0 0"/>
+            <geometry>
+                <box size="0.2 0.2 0.05"/>
+            </geometry>
+            <material name="grey">
+                <color rgba="0.5 0.5 0.5 1.0"/>
+            </material>
+        </visual>
+        <collision>
+            <origin xyz="0 0 0" rpy="0 0 0"/>
+            <geometry>
+                <box size="0.2 0.2 0.05"/>
+            </geometry>
+        </collision>
+        <inertial>
+            <mass value="0.5"/>
+            <inertia ixx="0.001" ixy="0.0" ixz="0.0" iyy="0.001" iyz="0.0" izz="0.001"/>
+        </inertial>
+    </link>
+    <joint name="lifter_joint" type="prismatic">
+        <parent link="chassis"/> <child link="lifter_link"/>
+        <origin xyz="0 0 0.25" rpy="0 0 0"/>
+        <axis xyz="0 0 1"/>
+        <limit lower="0.0" upper="0.20" effort="100.0" velocity="0.5"/>
+    </joint>
     <!-- BACK CASTER WHEEL LINK -->
     <!-- <joint name="back_caster_wheel_joint" type="fixed">

File: src/warehouse_real_description/description/ros2_control.xacro (robot description, xacro)
@@ -7,4 +7,5 @@
                 <param name="left_wheel_name">left_wheel_joint</param>
                 <param name="right_wheel_name">right_wheel_joint</param>
+                <param name="stepper_joint_name">lifter_joint</param>
                 <param name="loop_rate">30</param>
                 <param name="device">/dev/ttyACM0</param>
@@ -28,4 +29,11 @@
                 <state_interface name="position"/>
                 <state_interface name="velocity"/>
+            </joint>
+            <joint name="lifter_joint">
+                <command_interface name="position">
+                    <param name="min">0.0</param>
+                    <param name="max">0.20</param>
+                </command_interface>
+                <state_interface name="position"/>
             </joint>
         </ros2_control>
@@ -52,4 +60,11 @@
                 <state_interface name="position"/>
             </joint>
+            <joint name="lifter_joint">
+                <command_interface name="position">
+                    <param name="min">0.0</param>
+                    <param name="max">0.20</param>
+                </command_interface>
+                <state_interface name="position"/>
+            </joint>
         </ros2_control>
     </xacro:if>

Commit message: Editing urdf files to match real dimentions

File: src/warehouse_real_description/description/robot_core.xacro (robot description, xacro)
@@ -6,9 +6,9 @@
     <xacro:property name="chassis_height" value="0.15"/>
     <xacro:property name="chassis_mass" value="30.0"/>
-    <xacro:property name="wheel_radius" value="0.05"/>
+    <xacro:property name="wheel_radius" value="0.0625"/>
     <xacro:property name="wheel_thickness" value="0.02"/>
     <xacro:property name="wheel_mass" value="0.5"/>
     <xacro:property name="wheel_offset_x" value="0"/>
-    <xacro:property name="wheel_offset_y" value="${chassis_width/2 + wheel_thickness/2}"/>
+    <xacro:property name="wheel_offset_y" value="0.25"/>
     <xacro:property name="wheel_offset_z" value="${wheel_radius - (caster_wheel_radius*2)}"/>
     <xacro:property name="caster_wheel_radius" value="${0.03/2.0}"/>
